File: showcase/returnfrom.space/Hardware/supply.kicad_sch (KiCad schematic)
At the start: 8 parts, among them J1 USB_C_Receptacle_USB2.0_16P, U4 MT3608

Commit message: added step files
Parts:
- added J23: Conn_01x03_Pin, Connector_PinHeader_2.54mm:PinHeader_1x03_P2.54mm_Vertical, symbol Connector:Conn_01x03_Pin
- added R23: 5K1, Resistor_SMD:R_0402_1005Metric, symbol Device:R
- added U9: ~, spacescape:2xAA, symbol spacescape:2xAA
Connections:
- net GND: now also U9.-
- net at U4.5 (IN): now also J23.1 (Pin_1)
- new net: J23.2 (Pin_2), U9.+ (+3V)
- new net: J23.3 (Pin_3), R23.1
- new net BAT_TEST: R23.2
Other:
- moved on the sheet: U4

Commit message: updated
Parts:
- removed C1: 22uF, Capacitor_SMD:C_0805_2012Metric, symbol Device:C
- removed C2, C3: 100nF, Capacitor_SMD:C_0402_1005Metric, symbol Device:C
- removed J1: USB_C_Receptacle_USB2.0_16P, Connector_USB:USB_C_Receptacle_HCTL_HC-TYPE-C-16P-01A, symbol Connector:USB_C_Receptacle_USB2.0_16P
- removed J23: Conn_01x03_Pin, Connector_PinHeader_2.54mm:PinHeader_1x03_P2.54mm_Vertical, symbol Connector:Conn_01x03_Pin
- removed R1, R2, R23, R3: 5K1, Resistor_SMD:R_0402_1005Metric, symbol Device:R
- removed U4: MT3608, Package_TO_SOT_SMD:SOT-23-6, symbol Regulator_Switching:MT3608
- removed U9: ~, spacescape:2xAA, symbol spacescape:2xAA
Other:
- note removed: "request 5V/3A"
