File: showcase/returnfrom.space/Hardware/amp.kicad_sch (KiCad schematic)
At the start: 1 part, among them U5 LM324

Commit message: updated
Parts:
- added C27, C34: 100n, Capacitor_SMD:C_0402_1005Metric, symbol Device:C
- added C29, C30, C31, C33: 4u7, Capacitor_SMD:C_0402_1005Metric, symbol Device:C
- added C32: 33p, Capacitor_SMD:C_0402_1005Metric, symbol Device:C
- added D1: BP104-SMD, OptoDevice:Osram_BP104-SMD, symbol Sensor_Optical:BP104-SMD
- added MK2: Microphone, Sensor_Audio:CUI_CMC-4013-SMT, symbol Device:Microphone
- added R26, R27, R28, R31, R34: 10k, Resistor_SMD:R_0402_1005Metric, symbol Device:R
- added R29: 1k, Resistor_SMD:R_0402_1005Metric, symbol Device:R
- added R30, R32, R33, R35, R36: 100k, Resistor_SMD:R_0402_1005Metric, symbol Device:R
- added RV2: R_Potentiometer, Potentiometer_SMD:Potentiometer_Bourns_TC33X_Vertical, symbol Device:R_Potentiometer
Connections:
- net at U5.1: now also R29.2
- net at U5.2 (-): now also D1.1 (K), R28.1
- net at U5.3 (+): now also RV2.2
- net GND: now reaches U5.11 (V-)
- net GND: now also C27.2, C29.2, C31.2, C34.2, D1.2 (A), MK2.1 (-), R27.1, R33.1, R36.1
- net +5V: now reaches U5.4 (V+)
- net +5V: now also C27.1, R26.2, R28.2
- net at U5.5 (+): now also C33.2, R32.1, R33.2
- net at U5.6 (-): now also C32.1, R30.1, R31.2
- net at U5.7: now also C30.1, C32.2, R30.2
- new net: C33.1, C34.1, MK2.2 (+), R34.1
- new net: C29.1, C31.1, R31.1
- new net: R26.1, RV2.1
- new net: R27.2, RV2.3
- new net +3V3: R32.2, R34.2, R35.2
- new net ADC: C30.2, R35.1, R36.2
- new net GPIO: R29.1
Other:
- moved on the sheet: U5A, U5B, U5C, U5D, U5E

Commit message: updated
Parts:
- removed C31: 4u7, Capacitor_SMD:C_0402_1005Metric, symbol Device:C
- added RV1: R_Potentiometer_Trim, Potentiometer_SMD:Potentiometer_Bourns_TC33X_Vertical, symbol Device:R_Potentiometer_Trim
- C29, C30, C33: value 4u7 -> 22uF; footprint Capacitor_SMD:C_0402_1005Metric -> Capacitor_SMD:C_0805_2012Metric
- C32: value 33p -> 15pF
- R30, R32, R33: value 100k -> 47K
- R31, R34: value 10k -> 5K1
Connections:
- net +3V3: now also R34.1; no longer R34.2
- net GND: now also R33.2; no longer R33.1
- net at C33.2, R32.1, U5.5 (+): now also R33.1; no longer R33.2
- net at C33.1, C34.1, MK2.2 (+): now also R34.2; no longer R34.1
- net at R31.1: now also C32.1, R30.1, U5.6 (-); no longer C29.1
- new net: C29.1, R31.2
Other:
- moved on the sheet: C27, C34, D1, MK2, R26, R27, R28, R29, R35, R36, RV2, U5A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

Commit message: board almost done
Parts:
- removed RV1: R_Potentiometer_Trim, Potentiometer_SMD:Potentiometer_Bourns_TC33X_Vertical, symbol Device:R_Potentiometer_Trim
Changed lines of the file:
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@@
-	)
-	(symbol
-		(lib_id "Device:R_Potentiometer_Trim")
-		(at 139.7 128.27 0)
-		(mirror y)
-		(unit 1)
-		(exclude_from_sim no)
-		(in_bom yes)
-		(on_board yes)
-		(dnp no)
-		(fields_autoplaced yes)
-		(property "Reference" "RV1"
-			(at 142.24 126.9999 0)
-			(effects
-				(font
-					(size 1.27 1.27)
-				)
-				(justify right)
-			)
-		)
-		(property "Value" "R_Potentiometer_Trim"
-			(at 142.24 129.5399 0)
-			(effects
-				(font
-					(size 1.27 1.27)
-				)
-				(justify right)
-				(hide yes)
-			)
-		)
-		(property "Footprint" "Potentiometer_SMD:Potentiometer_Bourns_TC33X_Vertical"
-			(at 139.7 128.27 0)
-			(effects
-				(font
-					(size 1.27 1.27)
-				)
-				(hide yes)
-			)
-		)
-		(property "Datasheet" "~"
-			(at 139.7 128.27 0)
-			(effects
-				(font
-					(size 1.27 1.27)
-				)
-				(hide yes)
-			)
-		)
-		(property "Description" "Trim-potentiometer"
-			(at 139.7 128.27 0)
-			(effects
-				(font
-					(size 1.27 1.27)
-				)
-				(hide yes)
-			)
-		)
-		(pin "3"
-		)
-		(pin "2"
-		)
-		(pin "1"
-		)
-		(instances
-			(project "spacescape"
-				(path "/418a52ba-b136-48f0-a485-149e9dc1363e/7905eb6b-5a1a-4913-8ee0-ec6b3fb0933a"
-					(reference "RV1")
-					(unit 1)
-				)
-			)
-		)
 	)
 	(symbol

Commit message: panelizing...
Parts:
- removed D1: BP104-SMD, OptoDevice:Osram_BP104-SMD, symbol Sensor_Optical:BP104-SMD
- removed MK2: Microphone, Sensor_Audio:CUI_CMC-4013-SMT, symbol Device:Microphone
- removed U5: LM324, Package_DIP:DIP-14_W7.62mm_LongPads, symbol Amplifier_Operational:LM324
- added C79, C80: 1uF, Capacitor_SMD:C_0402_1005Metric, symbol Device:C
- added R107: 1K, Resistor_SMD:R_0402_1005Metric, symbol Device:R
- added RV8: R_Potentiometer, Potentiometer_THT:Potentiometer_Runtron_RM-065_Vertical, symbol Device:R_Potentiometer
- added U16: LMA3722T421-OA5, spacescape:LMA3722T421, symbol spacescape:LMA3722T421
- added U5: TLV2372, Package_SO:SOIC-8_3.9x4.9mm_P1.27mm, symbol Amplifier_Operational:TLV2372
- C27, C34: value 100n -> 1uF
- C29, C30, C33: value 22uF -> 1uF; footprint Capacitor_SMD:C_0805_2012Metric -> Capacitor_SMD:C_0402_1005Metric
- C32: value 15pF -> 1uF
- R26, R27, R28: value 10k -> 47K
- R29: value 1k -> 47K
- R31, R34: value 5K1 -> 47K
- R35, R36: value 100k -> 47K
- RV9: renamed from RV2; footprint Potentiometer_SMD:Potentiometer_Bourns_TC33X_Vertical -> Potentiometer_THT:Potentiometer_Runtron_RM-065_Vertical
Connections:
- net +3V3: now also C33.2, C34.1, R27.2, R29.2, C80.1, R107.1, U5.8 (V+)
- net GND: now also C33.1, R28.1, R31.2, C79.1, U16.3 (GND), U16.4 (GND), U5.4 (V-); no longer C27.2, C29.2, C34.2, R27.1
- net at C30.1, R30.2: now also U5.1; no longer C32.2
- net at C29.1: now also R26.2, U5.7; no longer R31.2
- net at R32.1, R33.1: now also C80.2, U5.3 (+); no longer C33.2
- net at R26.1: now also RV8.1, U5.6 (-); no longer RV9.1
- net at RV9.2: now also C27.2, RV9.3
- removed net +5V: C27.1, R26.2, R28.2
- net ADC renamed ADC2
- net GPIO: no longer names the net of R29.1
- net GPIO: now also C34.2, R31.1, U5.5 (+)
- new net: C79.2, R107.2, U16.2 (VDD)
- new net: C27.1, U16.1 (OUT)
- new net: R30.1, RV9.1, U5.2 (-)
- new net: C32.2, RV8.2, RV8.3
- new net ADC1: C29.2, R27.1, R28.2
- new net LDR: C32.1, R34.2
Other:
- moved on the sheet: R30, R32, R33, RV9
