File: showcase/returnfrom.space/Hardware/comms.kicad_sch (KiCad schematic)
At the start: 1 part

Commit message: panelizing...
Parts:
- removed MK1: Microphone, Sensor_Audio:POM-2244P-C3310-2-R, symbol Device:Microphone
Changed lines of the file:
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@@
 	(generator_version "9.0")
 	(paper "A4")
-	(symbol
-		(lib_id "Device:Microphone")
-		(at 85.09 110.49 0)
-		(unit 1)
-		(exclude_from_sim no)
-		(in_bom yes)
-		(on_board yes)
-		(dnp no)
-		(fields_autoplaced yes)
-		(property "Reference" "MK1"
-			(at 88.9 108.5214 0)
-			(effects
-				(font
-					(size 1.27 1.27)
-				)
-				(justify left)
-			)
-		)
-		(property "Value" "Microphone"
-			(at 88.9 111.0614 0)
-			(effects
-				(font
-					(size 1.27 1.27)
-				)
-				(justify left)
-			)
-		)
-		(property "Footprint" "Sensor_Audio:POM-2244P-C3310-2-R"
-			(at 85.09 107.95 90)
-			(effects
-				(font
-					(size 1.27 1.27)
-				)
-			)
-		)
-		(property "Datasheet" "~"
-			(at 85.09 107.95 90)
-			(effects
-				(font
-					(size 1.27 1.27)
-				)
-				(hide yes)
-			)
-		)
-		(property "Description" "Microphone"
-			(at 85.09 110.49 0)
-			(effects
-				(font
-					(size 1.27 1.27)
-				)
-				(hide yes)
-			)
-		)
-		(pin "1"
-		)
-		(pin "2"
-		)
-		(instances
-			(project "spacescape"
-				(path "/418a52ba-b136-48f0-a485-149e9dc1363e/f8071adf-8c79-49d8-9fd8-09b7aea99222"
-					(reference "MK1")
-					(unit 1)
-				)
-			)
-		)
-	)
 )
