File: showcase/returnfrom.space/Hardware/motherboard.kicad_sch (KiCad schematic)
At the start: 2 parts, among them J3 OLED, U2 ESP32-S2-SOLO

Commit message: added step files
Parts:
- J3: footprint Connector_PinSocket_2.54mm:PinSocket_1x04_P2.54mm_Vertical -> TG9541:Display_128x64_096_I2C
Changed lines of the file:
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@@
 			)
 		)
-		(property "Footprint" "Connector_PinSocket_2.54mm:PinSocket_1x04_P2.54mm_Vertical"
+		(property "Footprint" "TG9541:Display_128x64_096_I2C"
 			(at 165.1 39.37 0)
 			(effects

Commit message: updated
Parts:
- added C1, C37, C38, C40, C41: 22uF, Capacitor_SMD:C_0805_2012Metric, symbol Device:C
- added C2, C3: 100nF, Capacitor_SMD:C_0402_1005Metric, symbol Device:C
- added C42: 1uF, Capacitor_SMD:C_0402_1005Metric, symbol Device:C
- added D14: D, Diode_SMD:D_SOD-323, symbol Device:D
- added J1: USB_C_Receptacle_USB2.0_16P, Connector_USB:USB_C_Receptacle_HCTL_HC-TYPE-C-16P-01A, symbol Connector:USB_C_Receptacle_USB2.0_16P
- added L2: 4.7uH, Inductor_SMD:L_Changjiang_FNR4026S, symbol Device:L
- added R1, R2, R3, R44, R45, R46: 5K1, Resistor_SMD:R_0402_1005Metric, symbol Device:R
- added R23, R47, R48: 47K, Resistor_SMD:R_0402_1005Metric, symbol Device:R
- added R40, R41, R42, R43: 1K, Resistor_SMD:R_0402_1005Metric, symbol Device:R
- added SW19, SW20, SW21, SW22: SW_SPST, Button_Switch_SMD:SW_SPST_TL3305C, symbol Switch:SW_SPST
- added SW23: SW_SPDT_321, Button_Switch_THT:SW_Slide_SPDT_Angled_CK_OS102011MA1Q, symbol Switch:SW_SPDT_321
- added U10: AMS1117-3.3, Package_TO_SOT_SMD:SOT-223-3_TabPin2, symbol Regulator_Linear:AMS1117-3.3
- added U11: ~, spacescape:2xAA, symbol spacescape:2xAA
- added U4: MT3608L, Package_TO_SOT_SMD:SOT-23-6, symbol spacescape:MT3608L
Connections:
- net GND: now also C1.2, C2.2, C3.2, C37.2, C38.2, C40.2, C41.2, C42.2, J1.A1 (GND), J1.A12 (GND), J1.B1 (GND), J1.B12 (GND), R1.1, R2.1, R23.2, R3.2, R44.1, R46.1, SW19.2 (B), SW20.2 (B), SW21.2 (B), SW22.2 (B), U10.1 (GND), U11.-, U4.2 (GND)
- net at U2.13 (GPIO19/U1RTS/ADC2_CH8/CLK_OUT2/USB_D-): now also J1.A7 (D-), J1.B7 (D-)
- net at U2.14 (GPIO20/U1CTS/ADC2_CH9/CLK_OUT1/USB_D+): now also J1.A6 (D+), J1.B6 (D+)
- net K1: now reaches U2.4 (GPIO4/TOUCH4/ADC1_CH3)
- net K1: now also R40.1
- net K2: now reaches U2.5 (GPIO5/TOUCH5/ADC1_CH4)
- net K2: now also R41.1
- net K3: now reaches U2.6 (GPIO6/TOUCH6/ADC1_CH5)
- net K3: now also R42.1
- net K4: now reaches U2.7 (GPIO7/TOUCH7/ADC1_CH6)
- net K4: now also R43.1
- new net: R41.2, SW20.1 (A)
- new net: R46.2, R47.1, R48.1, U4.3 (FB)
- new net: C3.1, J1.S1 (SHIELD), R3.1
- new net: J1.A5 (CC1), R1.2
- new net: J1.B5 (CC2), R2.2
- new net: R23.1, U4.6 (OC)
- new net: R44.2, SW23.3 (A)
- new net: R42.2, SW21.1 (A)
- new net: D14.2 (A), L2.2, U4.1 (SW)
- new net: SW23.2 (B), U4.4 (EN)
- new net: C41.1, L2.1, R45.1, U11.+ (+3V), U4.5 (IN)
- new net: R43.2, SW22.1 (A)
- new net: R45.2, SW23.1 (C)
- new net: R40.2, SW19.1 (A)
- new net +3V3: C37.1, C38.1, C40.1, C42.1, D14.1 (K), R47.2, R48.2, U10.2 (VO)
- new net +5V: C1.1, C2.1, J1.A4 (VBUS), J1.A9 (VBUS), J1.B4 (VBUS), J1.B9 (VBUS), U10.3 (VI)
Other:
- note added: "request 5V/3A"
- moved on the sheet: J3

Commit message: updated
Parts:
- removed R40, R41, R42, R43: 1K, Resistor_SMD:R_0402_1005Metric, symbol Device:R
- removed SW19, SW20, SW21, SW22: SW_SPST, Button_Switch_SMD:SW_SPST_TL3305C, symbol Switch:SW_SPST
- removed U10: AMS1117-3.3, Package_TO_SOT_SMD:SOT-223-3_TabPin2, symbol Regulator_Linear:AMS1117-3.3
- removed U2: ESP32-S2-SOLO, Espressif:ESP32-S2-SOLO, symbol Espressif:ESP32-S2-SOLO
- added C31, C43: 1uF, Capacitor_SMD:C_0402_1005Metric, symbol Device:C
- added C44, C45: 22uF, Capacitor_SMD:C_0805_2012Metric, symbol Device:C
- added C46, C47: 100nF, Capacitor_SMD:C_0402_1005Metric, symbol Device:C
- added D15, D2: RED LED, LED_SMD:LED_0603_1608Metric, symbol Device:LED
- added D18: RED, LED_SMD:LED_0603_1608Metric, symbol Device:LED
- added D19: BLUE, LED_SMD:LED_0603_1608Metric, symbol Device:LED
- added J19: Conn_01x08_Pin, Connector_PinHeader_2.54mm:PinHeader_1x08_P2.54mm_Horizontal, symbol Connector:Conn_01x08_Pin
- added J2: Conn_01x08_Socket, Connector_FFC-FPC:TE_0-1734839-8_1x08-1MP_P0.5mm_Horizontal, symbol Connector:Conn_01x08_Socket
- added J5: 2x SERVO, Connector_PinHeader_2.54mm:PinHeader_2x03_P2.54mm_Vertical, symbol Connector_Generic:Conn_02x03_Odd_Even
- added L1: 2.2uH, Inductor_SMD:L_Cenker_CKCS201610, symbol Device:L
- added Q3: NPN, Package_TO_SOT_SMD:SOT-23, symbol Simulation_SPICE:NPN
- added R49, R61: 5K1, Resistor_SMD:R_0402_1005Metric, symbol Device:R
- added R50, R52, R53, R54, R57, R58, R63: 1K, Resistor_SMD:R_0402_1005Metric, symbol Device:R
- added R59, R62: 47K, Resistor_SMD:R_0402_1005Metric, symbol Device:R
- added R60: 215K, Resistor_SMD:R_0402_1005Metric, symbol Device:R
- added SW0: SW_SPST, Button_Switch_THT:SW_PUSH-12mm, symbol Switch:SW_SPST
- added SW24: SW_SPDT_321, Button_Switch_THT:SW_Slide_SPDT_Angled_CK_OS102011MA1Q, symbol Switch:SW_SPDT_321
- added SW25: BOOTSEL, Button_Switch_SMD:SW_SPST_TL3305C, symbol Switch:SW_SPST
- added U10: TLV62565DBVx, Package_TO_SOT_SMD:SOT-23-5, symbol Regulator_Switching:TLV62565DBVx
- added U6: TP4056, Package_SO:SOIC-8-1EP_3.9x4.9mm_P1.27mm_EP2.41x3.3mm_ThermalVias, symbol Battery_Management:TP4056-42-ESOP8
- added U9: ESP32-S2-MINI-2, Espressif:ESP32-S2-MINI-1, symbol Espressif:ESP32-S2-MINI-1
- L2: value 4.7uH -> 10uH; footprint Inductor_SMD:L_Changjiang_FNR4026S -> Inductor_SMD:L_APV_ANR4030
Connections:
- net +3V3: now also J3.2 (Pin_2), C31.2, C43.2, C47.2, J19.3 (Pin_3), J2.4 (Pin_4), L1.2, R49.1, R50.2, R53.1, R60.2, U9.3 (3V3); no longer C37.1
- net +5V: now also C37.1, D18.2 (A), D19.2 (A), J19.1 (Pin_1), R61.2, U6.4 (V_{CC}), U6.8 (CE)
- net GND: now also J3.1 (Pin_1), C31.1, C43.1, C44.2, C45.2, C46.1, C47.1, D15.1 (K), J19.4 (Pin_4), J2.6 (Pin_6), J5.1 (Pin_1), J5.2 (Pin_2), Q3.3 (E), R57.2, R59.1, R62.2, SW0.2 (B), SW25.2 (B), U10.2 (GND), U6.3 (GND), U6.9 (EPAD), U9.1 (GND), U9.2 (GND), U9.30 (GND), U9.42 (GND), U9.43 (GND), U9.46 (GND), U9.47 (GND), U9.48 (GND), U9.49 (GND), U9.50 (GND), U9.51 (GND), U9.52 (GND), U9.53 (GND), U9.54 (GND), U9.55 (GND), U9.56 (GND), U9.57 (GND), U9.58 (GND), U9.59 (GND), U9.60 (GND), U9.61 (GND), U9.62 (GND), U9.63 (GND), U9.64 (GND), U9.65 (GND)
- net K1: now also U9.16 (GPIO12/ADC2_CH1)
- net K2: now also U9.17 (GPIO13/ADC2_CH2)
- net K3: now also U9.18 (GPIO14/ADC2_CH3)
- net K4: now also U9.21 (ADC2_CH6/DAC_1/GPIO17)
- net at J1.A6 (D+), J1.B6 (D+): now also U9.24 (USB_D+/ADC2_CH9/GPIO20)
- net at J1.A7 (D-), J1.B7 (D-): now also U9.23 (USB_D-/ADC2_CH8/GPIO19)
- net EN2: now reaches SW23.2 (B), U4.4 (EN)
- net EN2: now also C46.2, Q3.1 (C)
- new net: D2.1 (K), J2.5 (Pin_5), R49.2, SW24.2 (B)
- new net: R52.1, SW0.1 (A), SW24.1 (C)
- new net: D15.2 (A), R53.2
- new net: R59.2, R60.1, U10.5 (FB)
- new net: L1.1, U10.3 (SW)
- new net: R57.1, U6.2 (PROG)
- new net: R58.1, R63.1, U6.6 (~{STDBY})
- new net: R54.2, U6.7 (~{CHRG})
- new net: Q3.2 (B), R61.1, R62.1
- new net: D18.1 (K), R54.1
- new net: D19.1 (K), R58.2, R63.2
- new net: D2.2 (A), R50.1
- new net +BATT: C44.1, C45.1, J5.3 (Pin_3), J5.4 (Pin_4), U10.1 (EN), U10.4 (VIN), U6.5 (BAT)
- new net ACC_INT: J2.1 (Pin_1)
- new net BOOT2: SW25.1 (A), U9.4 (GPIO0/BOOT)
- new net LASER_BTN: R52.2
- new net LASER_EN: SW24.3 (A)
- new net PHOTO1: J2.7 (Pin_7)
- new net PHOTO2: J2.8 (Pin_8)
- new net RST1: J19.2 (Pin_2)
- new net SCL: J2.3 (Pin_3)
- new net SDA: J2.2 (Pin_2)
- new net SERVO1: J5.5 (Pin_5), U9.6 (GPIO2/ADC1_CH1)
- new net SERVO2: J5.6 (Pin_6), U9.5 (GPIO1/ADC1_CH0)
- no-connect marks 0 -> 1
Other:
- note added: "2xAA BATTERY STEP-UP TO 3.3V"
- note added: "LASER MODULE CONTROL"
- note added: "LITHIUM BATTERY CHARGER"
- note added: "LITHIUM BATTERY STEP-DOWN TO 3.3V"
- note added: "OFF"
- note added: "ON"
- note added: "USB POWER + DATA"
- note added: "~3.344V"
- moved on the sheet: C1, C2, C3, C40, C41, C42, D14, J1, J3, L2, R1, R2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

Commit message: board almost done
Parts:
- removed J5: 2x SERVO, Connector_PinHeader_2.54mm:PinHeader_2x03_P2.54mm_Vertical, symbol Connector_Generic:Conn_02x03_Odd_Even
- added J4, J5: Conn_02x04_Odd_Even, Connector_PinHeader_2.54mm:PinHeader_2x04_P2.54mm_Vertical, symbol Connector_Generic:Conn_02x04_Odd_Even
- added R100, R101: 5K1, Resistor_SMD:R_0402_1005Metric, symbol Device:R
- added R67, R68, R96, R97, R98, R99: 27R, Resistor_SMD:R_0402_1005Metric, symbol Device:R
- added RXD2, TXD2: TestPoint, TestPoint:TestPoint_Pad_D2.0mm, symbol Connector:TestPoint
- renumbered R45 to R64, R44 to R65
Connections:
- net LASER_BTN is gone; now on net K7: R52.2
- net RST1 is gone; now on net IO11: J19.2 (Pin_2)
- net +3V3: now also J5.4 (Pin_4), R100.1, R101.2
- net +BATT: now also J4.1 (Pin_1), J4.5 (Pin_5), J4.6 (Pin_6)
- net GND: now also J4.4 (Pin_4), J5.2 (Pin_2)
- net K1: now also J5.6 (Pin_6)
- net K3: now also J5.1 (Pin_1)
- net K4: now also U9.19 (GPIO15/ADC2_CH4/XTAL_32K_P), J5.7 (Pin_7); no longer U9.21 (ADC2_CH6/DAC_1/GPIO17)
- net SERVO1: now also J4.7 (Pin_7)
- net SERVO2: now also J4.8 (Pin_8)
- net at J1.A6 (D+), J1.B6 (D+): now also R67.1; no longer U9.24 (USB_D+/ADC2_CH9/GPIO20)
- net at J1.A7 (D-), J1.B7 (D-): now also R68.1; no longer U9.23 (USB_D-/ADC2_CH8/GPIO19)
- net IO11: now reaches U9.15 (GPIO11/ADC2_CH0)
- net K5: now reaches U9.20 (GPIO16/ADC2_CH5/XTAL_32K_N)
- net K7: now reaches U9.22 (ADC2_CH7/DAC_2/GPIO18)
- net at U9.25 (GPIO21): now also R97.2
- net at U9.26 (SPI_CS1/GPIO26): now also R96.1
- net at U9.28 (GPIO33): now also R98.2
- net at U9.29 (GPIO34): now also R99.2
- net TXD2: now reaches U9.39 (GPIO43/U0TXD/PROG)
- net TXD2: now also TXD2.1
- net RXD2: now reaches U9.40 (GPIO44/U0RXD/PROG)
- net RXD2: now also RXD2.1
- net at J3.3 (Pin_3): now also R101.1
- net at J3.4 (Pin_4): now also R100.2
- net IO34: now reaches J19.5 (Pin_5)
- net IO34: now also R99.1
- net IO33: now reaches J19.6 (Pin_6)
- net IO33: now also R98.1
- net IO26: now reaches J19.7 (Pin_7)
- net IO26: now also R96.2
- net IO21: now reaches J19.8 (Pin_8)
- net IO21: now also R97.1
- new net: J4.2 (Pin_2), J4.3 (Pin_3)
- new net: R68.2, U9.23 (USB_D-/ADC2_CH8/GPIO19)
- new net: R67.2, U9.24 (USB_D+/ADC2_CH9/GPIO20)
- new net K6: U9.21 (ADC2_CH6/DAC_1/GPIO17)
Other:
- note added: "D-PAD CONNECTOR"
- note added: "NUMPAD"
- moved on the sheet: C31, C43, C44, D2, J19, J2, J3, R49, R50, R52, R57, SW0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

Commit message: panelizing...
Parts:
- added C89, C90, C91: 1uF, Capacitor_SMD:C_0402_1005Metric, symbol Device:C
- added C92: 100nF, Capacitor_SMD:C_0402_1005Metric, symbol Device:C
- added D25: D, Diode_SMD:D_SOD-323, symbol Device:D
- added IO3, IO4: TestPoint, TestPoint:TestPoint_Pad_D2.0mm, symbol Connector:TestPoint
- added J26: Conn_01x02, Connector_Hirose:Hirose_DF13-02P-1.25DS_1x02_P1.25mm_Horizontal, symbol Connector_Generic:Conn_01x02
- added J28: Conn_02x04_Odd_Even, Connector_PinHeader_2.54mm:PinHeader_2x04_P2.54mm_Vertical, symbol Connector_Generic:Conn_02x04_Odd_Even
- added R108: 27R, Resistor_SMD:R_0402_1005Metric, symbol Device:R
- added R121, R124, R125: 5K1, Resistor_SMD:R_0402_1005Metric, symbol Device:R
- added R122: 47K, Resistor_SMD:R_0402_1005Metric, symbol Device:R
- added R123: 1K, Resistor_SMD:R_0402_1005Metric, symbol Device:R
- added RV4: R_Potentiometer, Potentiometer_THT:Potentiometer_Runtron_RM-065_Vertical, symbol Device:R_Potentiometer
- added SW38: RESET, Button_Switch_SMD:SW_SPST_TL3305C, symbol Switch:SW_SPST
- added U19: FM8002, Package_SO:SOIC-8_3.9x4.9mm_P1.27mm, symbol spacescape:FM8002A
Connections:
- net ACC_INT is gone; now on net INT2: J2.1 (Pin_1)
- net IO21 is gone; now on net IO26: J19.8 (Pin_8), R97.1
- net PHOTO2 is gone; now on net GND: J2.8 (Pin_8)
- net SCL is gone; now on net SCL2: J2.3 (Pin_3)
- net SDA is gone; now on net SDA2: J2.2 (Pin_2)
- net +3V3: now also C91.2, R124.2, R125.1, U19.6 (VDD)
- net +5V: no longer R61.2
- net +BATT: now also D25.2 (A), J28.1 (Pin_1), J28.5 (Pin_5), J28.6 (Pin_6)
- net BOOT2: now also R124.1
- net GND: now also J4.2 (Pin_2), J4.3 (Pin_3), C90.2, C91.1, C92.2, J28.2 (Pin_2), J28.3 (Pin_3), J28.4 (Pin_4), R122.1, SW38.1 (A), U19.7 (GND)
- net IO26: no longer J19.7 (Pin_7), R96.2
- net K2: now also J5.8 (Pin_8)
- net K5: now also J5.5 (Pin_5), J28.8 (Pin_8)
- net K6: now also J5.3 (Pin_3), U9.9 (GPIO5/ADC1_CH4), J28.7 (Pin_7); no longer U9.21 (ADC2_CH6/DAC_1/GPIO17)
- net LASER_EN: now also U9.32 (GPIO36)
- net SCL2: now reaches J3.3 (Pin_3), R101.1
- net SCL2: now also U9.11 (GPIO7/ADC1_CH6)
- net at D2.1 (K), R49.2: now also R52.1, SW0.1 (A), SW24.1 (C), C92.1; no longer J2.5 (Pin_5), SW24.2 (B)
- net +3V0: now reaches C41.1, L2.1, R64.1, U11.+ (+3V), U4.5 (IN)
- net at U9.10 (GPIO6/ADC1_CH5): now also R96.2
- net SDA2: now reaches U9.12 (GPIO8/ADC1_CH7)
- net SDA2: now also J3.4 (Pin_4), R100.2
- net INT2: now reaches U9.13 (GPIO9/ADC1_CH8)
- net ADC1: now reaches U9.14 (GPIO10/ADC1_CH9)
- net at R97.2: now also U9.26 (SPI_CS1/GPIO26); no longer U9.25 (GPIO21)
- net IO6: now reaches R96.1
- net IO6: now also J19.7 (Pin_7); no longer U9.26 (SPI_CS1/GPIO26)
- net at U9.31 (GPIO35): now also R108.2
- net at U9.45 (CHIP/PU/RESET): now also R125.2, SW38.2 (B)
- net at U9.7 (GPIO3/ADC1_CH2): now also IO3.1
- net at U9.8 (GPIO4/ADC1_CH3): now also IO4.1
- net IO11 renamed ADC2
- net ADC2: no longer J19.2 (Pin_2)
- net PHOTO1 renamed LDR
- new net: C89.1, R121.1
- new net: J2.5 (Pin_5), SW24.2 (B)
- new net: C90.1, U19.2 (BYPS), U19.3 (IN+)
- new net: R121.2, R123.1, U19.4 (IN-)
- new net: J26.2 (Pin_2), RV4.2, RV4.3, U19.5 (VO1)
- new net: J26.1 (Pin_1), U19.8 (VO2)
- new net: D25.1 (K), R61.2
- new net: R123.2, RV4.1
- new net AMP_EN: R122.2, U19.1 (SHDN), U9.25 (GPIO21)
- new net DAC1: C89.2, U9.21 (ADC2_CH6/DAC_1/GPIO17)
- new net IO35: J19.2 (Pin_2), R108.1
- no-connect marks 1 -> 11
Other:
- note added: "SPEAKER AMPLIFIER"
- moved on the sheet: D2, J3, R49, R50, R52, R96, R97, SW0, SW24

Commit message: Done. Ordered 50pcs. TO DO: clean-up, add BOM & POS
Parts:
- removed Q3: NPN, Package_TO_SOT_SMD:SOT-23, symbol Simulation_SPICE:NPN
- added Q3: BC817, Package_TO_SOT_SMD:SOT-23, symbol Transistor_BJT:BC817
Connections:
- net EN2: now also Q3.3 (C)
- net GND: now also Q3.2 (E)
- net at R61.1, R62.1: now also Q3.1 (B)
Changed lines of the file:
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@@
 	)
 	(junction
-		(at 228.6 36.83)
-		(diameter 0)
-		(color 0 0 0 0)
-	)
-	(junction
 		(at 238.76 86.36)
 		(diameter 0)
@@
 	)
 	(junction
+		(at 190.5 130.81)
+		(diameter 0)
+		(color 0 0 0 0)
+	)
+	(junction
 		(at 154.94 177.8)
 		(diameter 0)
@@
 	)
 	(junction
-		(at 190.5 130.81)
-		(diameter 0)
-		(color 0 0 0 0)
-	)
-	(junction
 		(at 274.32 96.52)
 		(diameter 0)
@@
 	(wire
 		(pts
-			(xy 228.6 36.83) (xy 228.6 46.99)
+			(xy 228.6 34.29) (xy 228.6 46.99)
+		)
+		(stroke
+			(width 0)
+			(type default)
+		)
+	)
+	(wire
+		(pts
+			(xy 190.5 130.81) (xy 190.5 132.08)
 		)
 		(stroke
@@
 	(wire
 		(pts
-			(xy 228.6 36.83) (xy 229.87 36.83)
-		)
-		(stroke
-			(width 0)
-			(type default)
-		)
-	)
-	(wire
-		(pts
 			(xy 251.46 128.27) (xy 251.46 130.81)
 		)
@@
 	(wire
 		(pts
-			(xy 190.5 130.81) (xy 190.5 132.08)
+			(xy 190.5 129.54) (xy 190.5 130.81)
 		)
 		(stroke
@@
 	(wire
 		(pts
-			(xy 228.6 34.29) (xy 228.6 36.83)
-		)
-		(stroke
-			(width 0)
-			(type default)
-		)
-	)
-	(wire
-		(pts
 			(xy 143.51 175.26) (xy 163.83 175.26)
 		)
@@
 	(wire
 		(pts
-			(xy 190.5 129.54) (xy 190.5 130.81)
-		)
-		(stroke
-			(width 0)
-			(type default)
-		)
-	)
-	(wire
-		(pts
 			(xy 128.27 59.69) (xy 135.89 59.69)
 		)
@@
 		)
 	)
-	(global_label "VBAT"
-		(shape input)
-		(at 229.87 36.83 0)
-		(fields_autoplaced yes)
-		(effects
-			(font
-				(size 1.27 1.27)
-			)
-			(justify left)
-		)
-		(property "Intersheetrefs" "${INTERSHEET_REFS}"
-			(at 237.27 36.83 0)
-			(effects
-				(font
-					(size 1.27 1.27)
-				)
-				(justify left)
-				(hide yes)
-			)
-		)
-	)
 	(global_label "SERVO1"
 		(shape input)
@@
 		)
 		(property "Value" "+5V"
-			(at 146.812 65.532 0)
+			(at 152.4 64.516 0)
 			(effects
 				(font
@@
 	)
 	(symbol
+		(lib_id "Transistor_BJT:BC817")
+		(at 195.58 130.81 0)
+		(unit 1)
+		(exclude_from_sim no)
+		(in_bom yes)
+		(on_board yes)
+		(dnp no)
+		(property "Reference" "Q3"
+			(at 198.882 127 0)
+			(effects
+				(font
+					(size 1.27 1.27)
+				)
+				(justify left)
+			)
+		)
+		(property "Value" "BC817"
+			(at 198.12 144.018 0)
+			(effects
+				(font
+					(size 1.27 1.27)
+				)
+				(justify left)
+			)
+		)
+		(property "Footprint" "Package_TO_SOT_SMD:SOT-23"
+			(at 200.66 132.715 0)
+			(effects
+				(font
+					(size 1.27 1.27)
+					(italic yes)
+				)
+				(justify left)
+				(hide yes)
+			)
+		)
+		(property "Datasheet" "https://www.onsemi.com/pub/Collateral/BC818-D.pdf"
+			(at 195.58 130.81 0)
+			(effects
+				(font
+					(size 1.27 1.27)
+				)
+				(justify left)
+				(hide yes)
+			)
+		)
+		(property "Description" "0.8A Ic, 45V Vce, NPN Transistor, SOT-23"
+			(at 195.58 130.81 0)
+			(effects
+				(font
+					(size 1.27 1.27)
+				)
+				(hide yes)
+			)
+		)
+		(pin "3"
+		)
+		(pin "2"
+		)
+		(pin "1"
+		)
+		(instances
+			(project "spacescape"
+				(path "/418a52ba-b136-48f0-a485-149e9dc1363e/710b34da-2ff3-4b03-8183-b6a3c08c9c0f"
+					(reference "Q3")
+					(unit 1)
+				)
+			)
+		)
+	)
+	(symbol
 		(lib_id "power:GND")
 		(at 198.12 27.94 270)
@@
 	)
 	(symbol
-		(lib_id "Simulation_SPICE:NPN")
-		(at 195.58 130.81 0)
-		(unit 1)
-		(exclude_from_sim no)
-		(in_bom yes)
-		(on_board yes)
-		(dnp no)
-		(property "Reference" "Q3"
-			(at 193.294 126.746 0)
-			(effects
-				(font
-					(size 1.27 1.27)
-				)
-				(justify left)
-			)
-		)
-		(property "Value" "NPN"
-			(at 193.802 136.398 0)
-			(effects
-				(font
-					(size 1.27 1.27)
-				)
-				(justify left)
-			)
-		)
-		(property "Footprint" "Package_TO_SOT_SMD:SOT-23"
-			(at 259.08 130.81 0)
-			(effects
-				(font
-					(size 1.27 1.27)
-				)
-				(hide yes)
-			)
-		)
-		(property "Datasheet" "https://ngspice.sourceforge.io/docs/ngspice-html-manual/manual.xhtml#cha_BJTs"
-			(at 259.08 130.81 0)
-			(effects
-				(font
-					(size 1.27 1.27)
-				)
-				(hide yes)
-			)
-		)
-		(property "Description" "Bipolar transistor symbol for simulation only, substrate tied to the emitter"
-			(at 195.58 130.81 0)
-			(effects
-				(font
-					(size 1.27 1.27)
-				)
-				(hide yes)
-			)
-		)
-		(property "Sim.Device" "NPN"
-			(at 195.58 130.81 0)
-			(effects
-				(font
-					(size 1.27 1.27)
-				)
-				(hide yes)
-			)
-		)
-		(property "Sim.Type" "GUMMELPOON"
-			(at 195.58 130.81 0)
-			(effects
-				(font
-					(size 1.27 1.27)
-				)
-				(hide yes)
-			)
-		)
-		(property "Sim.Pins" "1=C 2=B 3=E"
-			(at 195.58 130.81 0)
-			(effects
-				(font
-					(size 1.27 1.27)
-				)
-				(hide yes)
-			)
-		)
-		(pin "3"
-		)
-		(pin "1"
-		)
-		(pin "2"
-		)
-		(instances
-			(project ""
-				(path "/418a52ba-b136-48f0-a485-149e9dc1363e/710b34da-2ff3-4b03-8183-b6a3c08c9c0f"
-					(reference "Q3")
-					(unit 1)
-				)
-			)
-		)
-	)
-	(symbol
 		(lib_id "Device:R")
 		(at 142.24 137.16 90)
@@
 		)
 		(property "Value" "GND"
-			(at 136.144 66.04 0)
+			(at 142.24 65.024 0)
 			(effects
 				(font
