File: showcase/returnfrom.space/Hardware/sigma/sigma.kicad_pcb (KiCad board)
At the start: 4 copper layers, 123 x 55 mm, 117 parts, among them J1 USB_C_Receptacle_USB2.0_16P, J19 Conn_01x08_Pin, J2 Conn_01x08_Socket, J26 Conn_01x02, J3 OLED, J4 Conn_02x03_Odd_Even, J5 Conn_02x04_Odd_Even, J6 Conn_02x03_Odd_Even, J7 Conn_01x02, Q3 BC817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

Commit message: sigma fix - not validated
Parts:
- added C15: 100uF, Capacitor_SMD:CP_Elec_6.3x5.4, F.Cu at (71.0, 71.0)
- added C16: 100uF, Capacitor_SMD:CP_Elec_6.3x5.4, F.Cu at (105.5, 40.0)
- added C17: 100uF, Capacitor_SMD:CP_Elec_6.3x5.4, F.Cu at (122.0, 56.0)
- added C18: 1uF, Capacitor_SMD:C_0402_1005Metric, F.Cu at (42.5, 56.6)
- added R8: DNP, Resistor_SMD:R_0402_1005Metric, B.Cu at (138.5, 39.9)
- added R9: DNP, Resistor_SMD:R_0402_1005Metric, B.Cu at (151.2, 41.2)
- J4, J6: footprint Connector_PinHeader_2.54mm:PinHeader_2x03_P2.54mm_Vertical -> Connector_PinHeader_2.54mm:PinHeader_2x03_P2.54mm_Horizontal
- moved J7 19.5 mm to (83.7, 68.0)
- moved J6 9.97 mm to (105.5, 45.6)
- moved R61 8.42 mm to (59.3, 64.4), turned to 0 degrees
- moved R62 8.26 mm to (59.3, 66.8), turned to 0 degrees
- moved D25 8.25 mm to (59.2, 62.0)
- moved J26 6.26 mm to (113.9, 50.4)
- moved Q3 5.77 mm to (59.5, 70.3)
- moved C11 4.87 mm to (61.6, 64.4)
- moved C41 4.87 mm to (63.7, 70.4)
- moved R5 4.87 mm to (61.6, 63.4)
- moved C10 4.87 mm to (63.0, 65.6)
- moved C42 4.87 mm to (63.5, 63.3)
- moved R4 4.87 mm to (60.6, 65.6)
- moved U1 4.87 mm to (62.0, 68.0)
- moved L2 4.87 mm to (62.3, 72.5)
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Routing:
- net LDR: track 71.7 -> 107.7 mm
- net /motherboard/K3: track 103.9 -> 120.5 mm
- net /motherboard/K4: track 97.3 -> 112.6 mm
- net /motherboard/K5: track 104.6 -> 119.6 mm
- net +BATT: track 104.2 -> 118.6 mm, vias 9 -> 12
- net /motherboard/K2: track 94.8 -> 108.4 mm
- net /motherboard/K6: track 117.7 -> 131.1 mm
- net /motherboard/K1: track 96.4 -> 106.7 mm
- net +3V3: track 51.3 -> 59.9 mm, vias 26 -> 33
- net Net-(J26-Pin_1): track 13.0 -> 7.10 mm
- net Net-(J26-Pin_2): track 24.2 -> 18.5 mm
- net /motherboard/EN2: track 20.8 -> 26.3 mm
- net +3V0: track 32.2 -> 37.3 mm
- net /motherboard/DAC1: track 84.4 -> 79.4 mm
- net ADC2: track 134.9 -> 139.8 mm
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Other:
- outline, holes or cut-outs redrawn
- board text added: "- -"
- board text added: "A"
- board text added: "BOOT"
- board text added: "Baterie Litiu"
- board text added: "C"
- board text added: "D"
- board text added: "NAVA SPAȚIALĂ SIGMA V1.1"
- board text added: "RST"
- board text removed: "PLACĂ DE BAZĂ SIGMA V1.1"
- board text removed: "R"
